Commit message: added joint in emerge_module

File: urdf/emerge_module.xacro (robot description, xacro)
@@ -6,5 +6,5 @@
         <origin xyz="0 0 0" rpy="0 0 0" />
         <geometry>
-          <box size="0.0305 0.0275 0.0385" />
+          <box size="0.0385 0.0305 0.0275" />
         </geometry>
         <material name="orange">
@@ -25,3 +25,4 @@
     </link>
   </xacro:macro>
+  <xacro:emerge_module name="emerge_module" />
 </robot>

File: urdf/flat_base.xacro (robot description, xacro)
@@ -1,43 +1,37 @@
 <?xml version="1.0"?>
 <robot xmlns:xacro="http://www.ros.org/wiki/xacro">
-    <xacro:macro name="flat_base" params="name='flat_base'">
-        <xacro:property name="name" value="flat_base" />
-        <xacro:property name="mass" value="0.65" /> <!-- kg -->
-        <xacro:property name="size_x" value="0.1494" />   <!-- meters -->
-        <xacro:property name="size_y" value="0.1494" />   <!-- meters -->
-        <xacro:property name="size_z" value="0.055023" /> <!-- meters -->
-        <!-- Inertia for a solid box -->
-        <xacro:property name="ixx" value="${(1.0/12.0) * mass * (size_y*size_y + size_z*size_z)}" />
-        <xacro:property name="iyy" value="${(1.0/12.0) * mass * (size_x*size_x + size_z*size_z)}" />
-        <xacro:property name="izz" value="${(1.0/12.0) * mass * (size_x*size_x + size_y*size_y)}" />
-        <link name="${name}_link">
-            <inertial>
-                <origin xyz="0 0 0" rpy="0 0 0" />
-                <mass value="${mass}" />
-                <inertia
-                    ixx="${ixx}" ixy="0.0" ixz="0.0"
-                    iyy="${iyy}" iyz="0.0"
-                    izz="${izz}" />
-            </inertial>
-            <visual>
-                <origin xyz="0 0 0" rpy="0 0 0" />
-                <geometry>
-                    <box size="0.0747 0.0747 0.0275115" />
-                </geometry>
-                <material name="grey">
-                    <color rgba="0.7 0.7 0.7 1.0" />
-                </material>
-            </visual>
-            <collision>
-                <origin xyz="0 0 0" rpy="0 0 0" />
-                <geometry>
-                    <box size="${size_x} ${size_y} ${size_z}" />
-                </geometry>
-            </collision>
-        </link>
-        <!-- =================== -->
-        <!-- Face frames (for modular connections) -->
-        <!-- =================== -->
-        <!-- Positions and normals from originFaceVector and normalFaceVector -->
-    </xacro:macro>
+  <xacro:macro name="flat_base" params="name='flat_base'">
+    <xacro:property name="name" value="flat_base"/>
+    <xacro:property name="mass" value="0.65"/>
+    <xacro:property name="size_x" value="0.1494"/>
+    <xacro:property name="size_y" value="0.1494"/>
+    <xacro:property name="size_z" value="0.055023"/>
+    <!-- Inertia for a solid box -->
+    <xacro:property name="ixx" value="${(1.0/12.0) * mass * (size_y*size_y + size_z*size_z)}"/>
+    <xacro:property name="iyy" value="${(1.0/12.0) * mass * (size_x*size_x + size_z*size_z)}"/>
+    <xacro:property name="izz" value="${(1.0/12.0) * mass * (size_x*size_x + size_y*size_y)}"/>
+    <link name="${name}_link">
+      <inertial>
+        <origin xyz="0 0 0" rpy="0 0 0"/>
+        <mass value="${mass}"/>
+        <inertia ixx="${ixx}" ixy="0.0" ixz="0.0" iyy="${iyy}" iyz="0.0" izz="${izz}"/>
+      </inertial>
+      <visual>
+        <origin xyz="0 0 0" rpy="0 0 0"/>
+        <geometry>
+          <box size="0.0747 0.0747 0.0275115"/>
+        </geometry>
+        <material name="grey">
+          <color rgba="0.7 0.7 0.7 1.0"/>
+        </material>
+      </visual>
+      <collision>
+        <origin xyz="0 0 0" rpy="0 0 0"/>
+        <geometry>
+          <box size="${size_x} ${size_y} ${size_z}"/>
+        </geometry>
+      </collision>
+    </link>
+  </xacro:macro>
+  <xacro:flat_base name="flat_base"/>
 </robot>

File: urdf/modular_robot.urdf (robot description, URDF)
Before this commit: robot modular_robot, 3 links, 2 joints
Links:
- removed link emerge_minus_link
- removed link emerge_plus_link
- added link emerge_minus_connector_link, mass 0.06; collision box size=0.061 0.055 0.077; visual box size=0.0385 0.0305 0.0275
- added link emerge_minus_motor_link, mass 0.06; collision box size=0.061 0.055 0.077; visual box size=0.048125 0.038125 0.034375
- added link emerge_plus_connector_link, mass 0.06; collision box size=0.061 0.055 0.077; visual box size=0.0385 0.0305 0.0275
- added link emerge_plus_motor_link, mass 0.06; collision box size=0.061 0.055 0.077; visual box size=0.048125 0.038125 0.034375
Joints:
- added joint emerge_minus_joint: type revolute, parent emerge_minus_connector_link, child emerge_minus_motor_link, origin xyz=0.03 0 0 rpy=0 0 0, axis 0 0 1, limit lower=-1.57 upper=1.57 effort=0.5 velocity=2.0
- added joint emerge_plus_joint: type revolute, parent emerge_plus_connector_link, child emerge_plus_motor_link, origin xyz=0.03 0 0 rpy=0 0 0, axis 0 0 1, limit lower=-1.57 upper=1.57 effort=0.5 velocity=2.0
- joint joint_x_minus: child emerge_minus_link -> emerge_minus_connector_link
- joint joint_x_plus: child emerge_plus_link -> emerge_plus_connector_link

File: urdf/modular_robot.urdf.xacro (robot description, xacro)
@@ -2,19 +2,18 @@
 <robot xmlns:xacro="http://www.ros.org/wiki/xacro" name="modular_robot">
   <!-- Include submodules -->
-  <xacro:include filename="emerge_module.xacro" />
-  <xacro:include filename="flat_base.xacro" />
-  <!-- Instantiate modules -->
-  <xacro:emerge_module name="emerge_plus" />
-  <xacro:emerge_module name="emerge_minus" />
-  <xacro:flat_base name="flat_base" />
+  <xacro:include filename="emerge_module2.xacro"/>
+  <xacro:include filename="flat_base.xacro"/>
+  <!-- Instantiate base and modules -->
+  <xacro:flat_base name="flat_base"/>
+  <xacro:emerge_module name="emerge_plus"/>
+  <xacro:emerge_module name="emerge_minus"/>
   <!-- Position properties -->
-  <!-- Using visual box dimensions to make surfaces touch -->
-  <xacro:property name="flat_half_x" value="${0.0747 / 2.0}" />
-  <xacro:property name="emerge_half_x" value="${0.0305 / 2.0}" />
-  <xacro:property name="joint_offset_x" value="${flat_half_x + emerge_half_x}" />
+  <xacro:property name="flat_half_x" value="${0.0747 / 2.0}"/>
+  <xacro:property name="emerge_half_x" value="${0.0305 / 2.0}"/>
+  <xacro:property name="joint_offset_x" value="${flat_half_x + emerge_half_x}"/>
   <!-- +X side -->
   <joint name="joint_x_plus" type="fixed">
     <parent link="flat_base_link"/>
-    <child link="emerge_plus_link"/>
+    <child link="emerge_plus_connector_link"/>
     <origin xyz="${joint_offset_x} 0 0" rpy="0 0 0"/>
   </joint>
@@ -22,5 +21,5 @@
   <joint name="joint_x_minus" type="fixed">
     <parent link="flat_base_link"/>
-    <child link="emerge_minus_link"/>
+    <child link="emerge_minus_connector_link"/>
     <origin xyz="${-1 * joint_offset_x} 0 0" rpy="0 0 ${pi}"/>
   </joint>

Commit message: added some control to the joints, a sinusoidal target like in edhmor

File: urdf/emerge_module.xacro (robot description, xacro)
@@ -1,28 +1,59 @@
 <?xml version="1.0"?>
-<robot xmlns:xacro="http://ros.org/wiki/xacro">
+<robot xmlns:xacro="http://www.ros.org/wiki/xacro">
+  <!-- Macro definition -->
   <xacro:macro name="emerge_module" params="name">
-    <link name="${name}_link">
+    <link name="${name}_connector_link">
       <visual>
-        <origin xyz="0 0 0" rpy="0 0 0" />
+        <origin xyz="0 0 0" rpy="0 0 0"/>
         <geometry>
-          <box size="0.0385 0.0305 0.0275" />
+          <box size="0.0385 0.0305 0.0275"/>
         </geometry>
         <material name="orange">
-          <color rgba="1 0.4 0 1" />
+          <color rgba="1 0.4 0 1"/>
         </material>
       </visual>
       <collision>
-        <origin xyz="0 0 0" rpy="0 0 0" />
+        <origin xyz="0 0 0" rpy="0 0 0"/>
         <geometry>
-          <box size="0.061 0.055 0.077" />
+          <box size="0.061 0.055 0.077"/>
         </geometry>
       </collision>
       <inertial>
-        <mass value="0.06" />
+        <origin xyz="0 0 0" rpy="0 0 0"/>
+        <mass value="0.06"/>
         <inertia ixx="0.00006" iyy="0.00005" izz="0.00007"
-          ixy="0" ixz="0" iyz="0" />
+                 ixy="0" ixz="0" iyz="0"/>
       </inertial>
     </link>
+    <link name="${name}_motor_link">
+      <visual>
+        <origin xyz="0 0 0" rpy="0 0 0"/>
+        <geometry>
+          <box size="0.048125 0.038125 0.034375"/>
+        </geometry>
+        <material name="orange">
+          <color rgba="1 0.4 0 1"/>
+        </material>
+      </visual>
+      <collision>
+        <origin xyz="0 0 0" rpy="0 0 0"/>
+        <geometry>
+          <box size="0.061 0.055 0.077"/>
+        </geometry>
+      </collision>
+      <inertial>
+        <origin xyz="0 0 0" rpy="0 0 0"/>
+        <mass value="0.06"/>
+        <inertia ixx="0.00006" iyy="0.00005" izz="0.00007"
+                 ixy="0" ixz="0" iyz="0"/>
+      </inertial>
+    </link>
+    <joint name="${name}_joint" type="revolute">
+      <parent link="${name}_connector_link"/>
+      <child link="${name}_motor_link"/>
+      <origin xyz="0.03 0 0" rpy="0 0 0"/>
+      <axis xyz="0 1 0"/>
+      <limit effort="0.5" velocity="2.0" lower="-0.12" upper="0.12"/>
+    </joint>
   </xacro:macro>
-  <xacro:emerge_module name="emerge_module" />
 </robot>

File: urdf/flat_base.xacro (robot description, xacro)
@@ -34,4 +34,3 @@
     </link>
   </xacro:macro>
-  <xacro:flat_base name="flat_base"/>
 </robot>

File: urdf/modular_robot.urdf (robot description, URDF)
Before this commit: robot modular_robot, 5 links, 4 joints
Joints:
- joint emerge_minus_joint: axis 0 0 1 -> 0 1 0; limit lower=-1.57 upper=1.57 effort=0.5 velocity=2.0 -> lower=-0.12 upper=0.12 effort=0.5 velocity=2.0
- joint emerge_plus_joint: axis 0 0 1 -> 0 1 0; limit lower=-1.57 upper=1.57 effort=0.5 velocity=2.0 -> lower=-0.12 upper=0.12 effort=0.5 velocity=2.0

File: urdf/modular_robot.urdf.xacro (robot description, xacro)
@@ -2,5 +2,5 @@
 <robot xmlns:xacro="http://www.ros.org/wiki/xacro" name="modular_robot">
   <!-- Include submodules -->
-  <xacro:include filename="emerge_module2.xacro"/>
+  <xacro:include filename="emerge_module.xacro"/>
   <xacro:include filename="flat_base.xacro"/>
   <!-- Instantiate base and modules -->

Commit message: joints move smoothly

File: urdf/emerge_module.xacro (robot description, xacro)
@@ -5,55 +5,57 @@
     <link name="${name}_connector_link">
       <visual>
-        <origin xyz="0 0 0" rpy="0 0 0"/>
+        <origin xyz="0 0 0" rpy="0 0 0" />
         <geometry>
-          <box size="0.0385 0.0305 0.0275"/>
+          <box size="0.0385 0.0305 0.0275" />
         </geometry>
         <material name="orange">
-          <color rgba="1 0.4 0 1"/>
+          <color rgba="1 0.4 0 1" />
         </material>
       </visual>
       <collision>
-        <origin xyz="0 0 0" rpy="0 0 0"/>
+        <origin xyz="0 0 0" rpy="0 0 0" />
         <geometry>
-          <box size="0.061 0.055 0.077"/>
+          <box size="0.0385 0.0305 0.0275" />
         </geometry>
       </collision>
       <inertial>
-        <origin xyz="0 0 0" rpy="0 0 0"/>
-        <mass value="0.06"/>
+        <origin xyz="0 0 0" rpy="0 0 0" />
+        <mass value="0.06" />
         <inertia ixx="0.00006" iyy="0.00005" izz="0.00007"
-                 ixy="0" ixz="0" iyz="0"/>
+          ixy="0" ixz="0" iyz="0" />
       </inertial>
     </link>
     <link name="${name}_motor_link">
       <visual>
-        <origin xyz="0 0 0" rpy="0 0 0"/>
+        <origin xyz="0 0 0" rpy="0 0 0" />
         <geometry>
-          <box size="0.048125 0.038125 0.034375"/>
+          <box size="0.048125 0.038125 0.034375" />
         </geometry>
         <material name="orange">
-          <color rgba="1 0.4 0 1"/>
+          <color rgba="1 0.4 0 1" />
         </material>
       </visual>
       <collision>
-        <origin xyz="0 0 0" rpy="0 0 0"/>
+        <origin xyz="0 0 0" rpy="0 0 0" />
         <geometry>
-          <box size="0.061 0.055 0.077"/>
+          <box size="0.048125 0.038125 0.034375" />
         </geometry>
       </collision>
       <inertial>
-        <origin xyz="0 0 0" rpy="0 0 0"/>
-        <mass value="0.06"/>
+        <origin xyz="0 0 0" rpy="0 0 0" />
+        <mass value="0.06" />
         <inertia ixx="0.00006" iyy="0.00005" izz="0.00007"
-                 ixy="0" ixz="0" iyz="0"/>
+          ixy="0" ixz="0" iyz="0" />
       </inertial>
     </link>
     <joint name="${name}_joint" type="revolute">
-      <parent link="${name}_connector_link"/>
-      <child link="${name}_motor_link"/>
-      <origin xyz="0.03 0 0" rpy="0 0 0"/>
-      <axis xyz="0 1 0"/>
-      <limit effort="0.5" velocity="2.0" lower="-0.12" upper="0.12"/>
+      <parent link="${name}_connector_link" />
+      <child link="${name}_motor_link" />
+      <origin xyz="0.03 0 0" rpy="0 0 0" />
+      <axis xyz="0 1 0" />
+      <!-- <limit effort="0.5" velocity="2.0" lower="-0.12" upper="0.12" /> -->
+       <limit effort="0.5" velocity="2.0" lower="-0.6" upper="0.6" />
     </joint>
   </xacro:macro>
+  <!-- <xacro:emerge_module name="emerge_plus"/> -->
 </robot>

File: urdf/modular_robot.urdf (robot description, URDF)
Before this commit: robot modular_robot, 5 links, 4 joints
Links:
- link emerge_minus_connector_link: geometry collision box size=0.0385 0.0305 0.0275; visual box size=0.0385 0.0305 0.0275
- link emerge_minus_motor_link: geometry collision box size=0.048125 0.038125 0.034375; visual box size=0.048125 0.038125 0.034375
- link emerge_plus_connector_link: geometry collision box size=0.0385 0.0305 0.0275; visual box size=0.0385 0.0305 0.0275
- link emerge_plus_motor_link: geometry collision box size=0.048125 0.038125 0.034375; visual box size=0.048125 0.038125 0.034375
Joints:
- joint emerge_minus_joint: limit lower=-0.12 upper=0.12 effort=0.5 velocity=2.0 -> lower=-0.6 upper=0.6 effort=0.5 velocity=2.0
- joint emerge_plus_joint: limit lower=-0.12 upper=0.12 effort=0.5 velocity=2.0 -> lower=-0.6 upper=0.6 effort=0.5 velocity=2.0
- joint joint_x_minus: axis (none) -> 0 1 0; limit (none) -> lower=-1.57 upper=1.57 effort=10 velocity=3; type fixed -> revolute
- joint joint_x_plus: axis (none) -> 0 1 0; limit (none) -> lower=-1.57 upper=1.57 effort=10 velocity=3; type fixed -> revolute
