Commit message: successfuly creates a robot with modules connecting to the base, orientation bugs connecting modules to each other. Also changed modular_robot.xacro to use the xacros, which were lost in a previous commit

File: urdf/emerge_module.xacro (robot description, xacro)
@@ -1,7 +1,11 @@
 <?xml version="1.0"?>
 <robot xmlns:xacro="http://www.ros.org/wiki/xacro">
-  <!-- Macro definition -->
-  <xacro:macro name="emerge_module" params="name">
+  <xacro:macro name="emerge_module" params="name xyz:='0 0 0' rpy:='0 0 0'">
     <link name="${name}_connector_link">
+      <inertial>
+        <origin xyz="0 0 0" />
+        <mass value="0.06" />
+        <inertia ixx="8.43e-06" ixy="0" ixz="0" iyy="1.12e-05" iyz="0" izz="1.21e-05" />
+      </inertial>
       <visual>
         <origin xyz="0 0 0" rpy="0 0 0" />
@@ -14,19 +18,18 @@
       </visual>
       <collision>
-        <origin xyz="0 0 0" rpy="0 0 0" />
+        <origin xyz="0 0 0" />
         <geometry>
           <box size="0.0385 0.0305 0.0275" />
         </geometry>
       </collision>
-      <inertial>
-        <origin xyz="0 0 0" rpy="0 0 0" />
-        <mass value="0.06" />
-        <inertia ixx="0.00006" iyy="0.00005" izz="0.00007"
-          ixy="0" ixz="0" iyz="0" />
-      </inertial>
     </link>
     <link name="${name}_motor_link">
+      <inertial>
+        <origin xyz="0 0 0" />
+        <mass value="0.06" />
+        <inertia ixx="1.32e-05" ixy="0" ixz="0" iyy="1.75e-05" iyz="0" izz="1.89e-05" />
+      </inertial>
       <visual>
-        <origin xyz="0 0 0" rpy="0 0 0" />
+        <origin xyz="0 0 0" />
         <geometry>
           <box size="0.048125 0.038125 0.034375" />
@@ -37,25 +40,20 @@
       </visual>
       <collision>
-        <origin xyz="0 0 0" rpy="0 0 0" />
+        <origin xyz="0 0 0" />
         <geometry>
           <box size="0.048125 0.038125 0.034375" />
         </geometry>
       </collision>
-      <inertial>
-        <origin xyz="0 0 0" rpy="0 0 0" />
-        <mass value="0.06" />
-        <inertia ixx="0.00006" iyy="0.00005" izz="0.00007"
-          ixy="0" ixz="0" iyz="0" />
-      </inertial>
     </link>
     <joint name="${name}_joint" type="revolute">
       <parent link="${name}_connector_link" />
       <child link="${name}_motor_link" />
-      <origin xyz="0.03 0 0" rpy="0 0 0" />
+      <!-- Offset increased to remove collision overlap -->
+      <origin xyz="0.042 0 0" rpy="0 0 0" />
       <axis xyz="0 1 0" />
-      <!-- <limit effort="0.5" velocity="2.0" lower="-0.12" upper="0.12" /> -->
-       <limit effort="0.5" velocity="2.0" lower="-0.6" upper="0.6" />
+      <limit effort="0.5" lower="-0.6" upper="0.6" velocity="2.0" />
+      <dynamics damping="0.03" />
     </joint>
   </xacro:macro>
-  <!-- <xacro:emerge_module name="emerge_plus"/> -->
+  <xacro:emerge_module name="emerge_plus"/>
 </robot>

File: urdf/flat_base.xacro (robot description, xacro)
@@ -2,32 +2,31 @@
 <robot xmlns:xacro="http://www.ros.org/wiki/xacro">
   <xacro:macro name="flat_base" params="name='flat_base'">
-    <xacro:property name="name" value="flat_base"/>
-    <xacro:property name="mass" value="0.65"/>
-    <xacro:property name="size_x" value="0.1494"/>
-    <xacro:property name="size_y" value="0.1494"/>
-    <xacro:property name="size_z" value="0.055023"/>
-    <!-- Inertia for a solid box -->
-    <xacro:property name="ixx" value="${(1.0/12.0) * mass * (size_y*size_y + size_z*size_z)}"/>
-    <xacro:property name="iyy" value="${(1.0/12.0) * mass * (size_x*size_x + size_z*size_z)}"/>
-    <xacro:property name="izz" value="${(1.0/12.0) * mass * (size_x*size_x + size_y*size_y)}"/>
-    <link name="${name}_link">
+    <xacro:property name="name" value="flat_base" />
+    <xacro:property name="mass" value="0.65" />
+    <xacro:property name="size_x" value="0.1494" />
+    <xacro:property name="size_y" value="0.1494" />
+    <xacro:property name="size_z" value="0.055023" />
+    <xacro:property name="ixx" value="${(1.0/12.0) * mass * (size_y*size_y + size_z*size_z)}" />
+    <xacro:property name="iyy" value="${(1.0/12.0) * mass * (size_x*size_x + size_z*size_z)}" />
+    <xacro:property name="izz" value="${(1.0/12.0) * mass * (size_x*size_x + size_y*size_y)}" />
+    <link name="flat_base_link">
       <inertial>
-        <origin xyz="0 0 0" rpy="0 0 0"/>
-        <mass value="${mass}"/>
-        <inertia ixx="${ixx}" ixy="0.0" ixz="0.0" iyy="${iyy}" iyz="0.0" izz="${izz}"/>
+        <origin xyz="0 0 0" rpy="0 0 0" />
+        <mass value="0.65" />
+        <inertia ixx="0.000342" ixy="0" ixz="0" iyy="0.000342" iyz="0" izz="0.000604" />
       </inertial>
       <visual>
-        <origin xyz="0 0 0" rpy="0 0 0"/>
+        <origin xyz="0 0 0" rpy="0 0 0" />
         <geometry>
-          <box size="0.0747 0.0747 0.0275115"/>
+          <box size="0.0747 0.0747 0.0275115" />
         </geometry>
         <material name="grey">
-          <color rgba="0.7 0.7 0.7 1.0"/>
+          <color rgba="0.7 0.7 0.7 1" />
         </material>
       </visual>
       <collision>
-        <origin xyz="0 0 0" rpy="0 0 0"/>
+        <origin xyz="0 0 0" rpy="0 0 0" />
         <geometry>
-          <box size="${size_x} ${size_y} ${size_z}"/>
+          <box size="0.0747 0.0747 0.0275115" />
         </geometry>
       </collision>

File: urdf/modular_robot.urdf.xacro (robot description, xacro)
@@ -1,146 +1,27 @@
-<?xml version="1.0" ?>
-<robot name="modular_robot">
-  <!-- ==================== BASE ==================== -->
-  <link name="flat_base_link">
-    <inertial>
-      <origin xyz="0 0 0" rpy="0 0 0"/>
-      <mass value="0.65"/>
-      <!-- Box inertia, size 0.0747 x 0.0747 x 0.0275115 -->
-      <inertia ixx="0.000342" ixy="0" ixz="0" iyy="0.000342" iyz="0" izz="0.000604"/>
-    </inertial>
-    <visual>
-      <origin xyz="0 0 0" rpy="0 0 0"/>
-      <geometry>
-        <box size="0.0747 0.0747 0.0275115"/>
-      </geometry>
-      <material name="grey">
-        <color rgba="0.7 0.7 0.7 1"/>
-      </material>
-    </visual>
-    <!-- Collision now matches visual (no unintended overlaps) -->
-    <collision>
-      <origin xyz="0 0 0" rpy="0 0 0"/>
-      <geometry>
-        <box size="0.0747 0.0747 0.0275115"/>
-      </geometry>
-    </collision>
-  </link>
-  <!-- ==================== +X CONNECTOR ==================== -->
-  <link name="emerge_plus_connector_link">
-    <inertial>
-      <origin xyz="0 0 0"/>
-      <mass value="0.06"/>
-      <!-- computed inertia -->
-      <inertia ixx="8.43e-06" ixy="0" ixz="0" iyy="1.12e-05" iyz="0" izz="1.21e-05"/>
-    </inertial>
-    <visual>
-      <origin xyz="0 0 0" rpy="0 0 0"/>
-      <geometry>
-        <box size="0.0385 0.0305 0.0275"/>
-      </geometry>
-      <material name="orange">
-        <color rgba="1 0.4 0 1"/>
-      </material>
-    </visual>
-    <collision>
-      <origin xyz="0 0 0"/>
-      <geometry>
-        <box size="0.0385 0.0305 0.0275"/>
-      </geometry>
-    </collision>
-  </link>
-  <link name="emerge_plus_motor_link">
-    <inertial>
-      <origin xyz="0 0 0"/>
-      <mass value="0.06"/>
-      <!-- computed inertia -->
-      <inertia ixx="1.32e-05" ixy="0" ixz="0" iyy="1.75e-05" iyz="0" izz="1.89e-05"/>
-    </inertial>
-    <visual>
-      <origin xyz="0 0 0"/>
-      <geometry>
-        <box size="0.048125 0.038125 0.034375"/>
-      </geometry>
-      <material name="orange">
-        <color rgba="1 0.4 0 1"/>
-      </material>
-    </visual>
-    <collision>
-      <origin xyz="0 0 0"/>
-      <geometry>
-        <box size="0.048125 0.038125 0.034375"/>
-      </geometry>
-    </collision>
-  </link>
-  <joint name="emerge_plus_joint" type="revolute">
-    <parent link="emerge_plus_connector_link"/>
-    <child link="emerge_plus_motor_link"/>
-    <!-- Offset increased to remove collision overlap -->
-    <origin xyz="0.045 0 0" rpy="0 0 0"/>
-    <axis xyz="0 1 0"/>
-    <limit effort="0.5" lower="-0.6" upper="0.6" velocity="2.0"/>
-    <dynamics damping="0.03"/>
-  </joint>
-  <!-- ==================== -X CONNECTOR (Mirrored) ==================== -->
-  <link name="emerge_minus_connector_link">
-    <inertial>
-      <origin xyz="0 0 0"/>
-      <mass value="0.06"/>
-      <inertia ixx="8.43e-06" ixy="0" ixz="0" iyy="1.12e-05" iyz="0" izz="1.21e-05"/>
-    </inertial>
-    <visual>
-      <geometry>
-        <box size="0.0385 0.0305 0.0275"/>
-      </geometry>
-      <material name="orange">
-        <color rgba="1 0.4 0 1"/>
-      </material>
-    </visual>
-    <collision>
-      <geometry>
-        <box size="0.0385 0.0305 0.0275"/>
-      </geometry>
-    </collision>
-  </link>
-  <link name="emerge_minus_motor_link">
-    <inertial>
-      <origin xyz="0 0 0"/>
-      <mass value="0.06"/>
-      <inertia ixx="1.32e-05" ixy="0" ixz="0" iyy="1.75e-05" iyz="0" izz="1.89e-05"/>
-    </inertial>
-    <visual>
-      <geometry>
-        <box size="0.048125 0.038125 0.034375"/>
-      </geometry>
-      <material name="orange">
-        <color rgba="1 0.4 0 1"/>
-      </material>
-    </visual>
-    <collision>
-      <geometry>
-        <box size="0.048125 0.038125 0.034375"/>
-      </geometry>
-    </collision>
-  </link>
-  <joint name="emerge_minus_joint" type="revolute">
-    <parent link="emerge_minus_connector_link"/>
-    <child link="emerge_minus_motor_link"/>
-    <!-- Same offset fix -->
-    <origin xyz="0.045 0 0" rpy="0 0 0"/>
-    <axis xyz="0 1 0"/>
-    <limit effort="0.5" lower="-0.6" upper="0.6" velocity="2.0"/>
-    <dynamics damping="0.03"/>
-  </joint>
-  <!-- ==================== ATTACH TO BASE ==================== -->
+<?xml version="1.0"?>
+<robot xmlns:xacro="http://www.ros.org/wiki/xacro" name="modular_robot">
+  <xacro:include filename="emerge_module.xacro" />
+  <xacro:include filename="flat_base.xacro" />
+  <xacro:property name="flat_half_x" value="${0.0747 / 2.0}" />
+  <xacro:property name="emerge_half_x" value="${0.0305 / 2.0}" />
+  <xacro:property name="base_offset" value="${flat_half_x + emerge_half_x}" />
+  <xacro:flat_base name="flat_base" />
+  <xacro:emerge_module name="emerge_plus" />
+  <xacro:emerge_module name="emerge_minus" />
+  <xacro:emerge_module name="emerge_y" />
   <joint name="joint_x_plus" type="fixed">
-    <parent link="flat_base_link"/>
-    <child link="emerge_plus_connector_link"/>
-    <!-- Adjusted to prevent contact penetration -->
-    <origin xyz="0.0576 0 0" rpy="0 0 0"/>
+    <parent link="flat_base_link" />
+    <child link="emerge_plus_connector_link" />
+    <origin xyz="${base_offset} 0 0" rpy="0 0 0" />
   </joint>
   <joint name="joint_x_minus" type="fixed">
-    <parent link="flat_base_link"/>
-    <child link="emerge_minus_connector_link"/>
-    <origin xyz="-0.0576 0 0" rpy="0 0 3.141592653589793"/>
+    <parent link="flat_base_link" />
+    <child link="emerge_minus_connector_link" />
+    <origin xyz="${-1 * base_offset} 0 0" rpy="0 0 ${pi}" />
+  </joint>
+  <joint name="joint_y" type="fixed">
+    <parent link="flat_base_link" />
+    <child link="emerge_y_connector_link" />
+    <origin xyz="0 ${base_offset} 0" rpy="0 0 ${pi/2}" />
   </joint>
 </robot>
