Commit message: changed naming of elements

File: urdf/base.xacro (robot description, xacro)
@@ -1,5 +1,5 @@
 <?xml version="1.0"?>
 <robot xmlns:xacro="http://www.ros.org/wiki/xacro">
-  <xacro:macro name="flat_base" params="name='flat_base'">
+  <xacro:macro name="base" params="name='base'">
     <xacro:property name="name" value="flat_base" />
     <xacro:property name="mass" value="0.65" />
@@ -10,5 +10,5 @@
     <xacro:property name="iyy" value="${(1.0/12.0) * mass * (size_x*size_x + size_z*size_z)}" />
     <xacro:property name="izz" value="${(1.0/12.0) * mass * (size_x*size_x + size_y*size_y)}" />
-    <link name="flat_base_link">
+    <link name="base_link">
       <inertial>
         <origin xyz="0 0 0" rpy="0 0 0" />

File: urdf/modular_robot.urdf.xacro (robot description, xacro)
@@ -1,26 +1,26 @@
 <?xml version="1.0"?>
 <robot xmlns:xacro="http://www.ros.org/wiki/xacro" name="modular_robot">
-  <xacro:include filename="emerge_module.xacro" />
-  <xacro:include filename="flat_base.xacro" />
+  <xacro:include filename="module.xacro" />
+  <xacro:include filename="base.xacro" />
   <xacro:property name="flat_half_x" value="${0.0747 / 2.0}" />
   <xacro:property name="emerge_half_x" value="${0.0305 / 2.0}" />
   <xacro:property name="base_offset" value="${flat_half_x + emerge_half_x}" />
-  <xacro:flat_base name="flat_base" />
-  <xacro:emerge_module name="emerge_plus" />
-  <xacro:emerge_module name="emerge_minus" />
-  <xacro:emerge_module name="emerge_y" />
+  <xacro:base name="base" />
+  <xacro:module name="plus" />
+  <xacro:module name="minus" />
+  <xacro:module name="y" />
   <joint name="joint_x_plus" type="fixed">
-    <parent link="flat_base_link" />
-    <child link="emerge_plus_connector_link" />
+    <parent link="base_link" />
+    <child link="plus_connector_link" />
     <origin xyz="${base_offset} 0 0" rpy="0 0 0" />
   </joint>
   <joint name="joint_x_minus" type="fixed">
-    <parent link="flat_base_link" />
-    <child link="emerge_minus_connector_link" />
+    <parent link="base_link" />
+    <child link="minus_connector_link" />
     <origin xyz="${-1 * base_offset} 0 0" rpy="0 0 ${pi}" />
   </joint>
   <joint name="joint_y" type="fixed">
-    <parent link="flat_base_link" />
-    <child link="emerge_y_connector_link" />
+    <parent link="base_link" />
+    <child link="y_connector_link" />
     <origin xyz="0 ${base_offset} 0" rpy="0 0 ${pi/2}" />
   </joint>

File: urdf/module.xacro (robot description, xacro)
@@ -1,5 +1,5 @@
 <?xml version="1.0"?>
 <robot xmlns:xacro="http://www.ros.org/wiki/xacro">
-  <xacro:macro name="emerge_module" params="name xyz:='0 0 0' rpy:='0 0 0'">
+  <xacro:macro name="module" params="name xyz:='0 0 0' rpy:='0 0 0'">
     <link name="${name}_connector_link">
       <inertial>
@@ -56,4 +56,4 @@
     </joint>
   </xacro:macro>
-  <xacro:emerge_module name="emerge_plus"/>
+  <!-- <xacro:emerge_module name="instance"/> -->
 </robot>
