Commit message: orientations corrected, the tree, translation to urdf  and simulation work

File: urdf/modular_robot.urdf.xacro (robot description, xacro)
@@ -21,7 +21,7 @@
   </joint>
   <joint name="joint_y" type="fixed">
-    <parent link="base_link" />
+    <parent link="minus_motor_link" />
     <child link="y_connector_link" />
-    <origin xyz="0 ${base_offset} 0" rpy="0 0 ${pi/2}" />
+    <origin xyz="0.038125 0 0" rpy="0 0 0" />
   </joint>
 </robot>

File: urdf/random_robot.urdf.xacro (robot description, xacro)
@@ -7,12 +7,18 @@
     <parent link="base_link"/>
     <child link="module_0_connector_link"/>
-    <origin xyz="0 -0.0526 0" rpy="0 0 -1.5707963267948966"/>
+    <origin xyz="0 0.0526 0" rpy="0 0 1.5707963267948966"/>
   </joint>
   <xacro:module name="module_0"/>
-  <joint name="joint_base_module_1" type="fixed">
-    <parent link="base_link"/>
+  <joint name="joint_module_0_module_1" type="fixed">
+    <parent link="module_0_motor_link"/>
     <child link="module_1_connector_link"/>
-    <origin xyz="0 0.0526 0" rpy="0 0 1.5707963267948966"/>
+    <origin xyz="0 0.038125 0" rpy="0 0 1.5707963267948966"/>
   </joint>
   <xacro:module name="module_1"/>
+  <joint name="joint_module_0_module_2" type="fixed">
+    <parent link="module_0_motor_link"/>
+    <child link="module_2_connector_link"/>
+    <origin xyz="0 -0.038125 0" rpy="0 0 -1.5707963267948966"/>
+  </joint>
+  <xacro:module name="module_2"/>
 </robot>
